Commit message: nothing

File: marm_description/urdf/arm_base.xacro (robot description, xacro)
@@ -339,8 +339,8 @@
                 <type>transmission_interface/SimpleTransmission</type>
                 <joint name="${joint_name}">
-                    <hardwareInterface>hardware_interface/PositionJointInterface</hardwareInterface>
+                    <hardwareInterface>hardware_interface/EffortJointInterface</hardwareInterface>
                 </joint>
                 <actuator name="${joint_name}_motor">
-                    <hardwareInterface>hardware_interface/PositionJointInterface</hardwareInterface>
+                    <hardwareInterface>hardware_interface/EffortJointInterface</hardwareInterface>
                     <mechanicalReduction>1</mechanicalReduction>
                 </actuator>

File: marm_description/urdf/arm_gazebo.xacro (robot description, xacro)
@@ -22,9 +22,9 @@
     <arm_base parent="bottom_link" xyz="0 0 0.02" rpy="0 0 0"/>
     <!-- kinect -->
-    <joint name="kinect_joint" type="fixed">
+    <!--joint name="kinect_joint" type="fixed">
         <origin xyz="0.1 0 0.8" rpy="0 ${75.0 * deg_to_rad} 0" />
         <parent link="base_link"/>
         <child link="kinect_link"/>
     </joint>
-    <xacro:kinect_camera prefix="kinect"/>
+    <xacro:kinect_camera prefix="kinect"/-->
 </robot>

Commit message: single arm

File: marm_description/urdf/arm_base.xacro (robot description, xacro)
@@ -339,8 +339,8 @@
                 <type>transmission_interface/SimpleTransmission</type>
                 <joint name="${joint_name}">
-                    <hardwareInterface>hardware_interface/EffortJointInterface</hardwareInterface>
+                    <hardwareInterface>hardware_interface/PositionJointInterface</hardwareInterface>
                 </joint>
                 <actuator name="${joint_name}_motor">
-                    <hardwareInterface>hardware_interface/EffortJointInterface</hardwareInterface>
+                    <hardwareInterface>hardware_interface/PositionJointInterface</hardwareInterface>
                     <mechanicalReduction>1</mechanicalReduction>
                 </actuator>
@@ -357,5 +357,5 @@
         <gazebo>
             <plugin name="gazebo_ros_control" filename="libgazebo_ros_control.so">
-                <robotNamespace>/arm2</robotNamespace>
+                <robotNamespace>/arm</robotNamespace>
             </plugin>
         </gazebo>

File: marm_description/urdf/arm_gazebo.xacro (robot description, xacro)
@@ -1,6 +1,6 @@
 <?xml version="1.0"?>
-<robot name="arm2" xmlns:xacro="http://www.ros.org/wiki/xacro">
+<robot name="arm" xmlns:xacro="http://www.ros.org/wiki/xacro">
     <xacro:include filename="$(find marm_description)/urdf/arm_base.xacro" />
-    <xacro:include filename="$(find marm_description)/urdf/kinect_gazebo.xacro" />
+    <!--xacro:include filename="$(find marm_description)/urdf/kinect_gazebo.xacro" /-->
     <xacro:property name="deg_to_rad" value="0.01745329251994329577"/>
     <link name="bottom_link">

File: marm_description/urdf/dual_arm.xacro (robot description, xacro)
@@ -5,8 +5,11 @@
     <xacro:property name="stand_length" value="0.4"/>
     <xacro:include filename="$(find marm_description)/urdf/arm_base_gazebo.xacro" />
-    <link name="virtual_link" />
-    <joint name="virtual_joint" type="fixed">
+    <link name="virtuallink" />
+    <gazebo reference="virtuallink">
+        <material>Gazebo/Gray</material>
+    </gazebo>
+    <joint name="virtualjoint" type="fixed">
         <origin xyz="0 0 0" rpy="0 0 0" />
-        <parnet link="virtual_link" />
+        <parent link="virtuallink" />
         <child link="base_link" />
     </joint>
