Commit message: marm

File: marm_description/urdf/marm.xacro (robot description, xacro)
@@ -9,7 +9,7 @@
     <xacro:include filename="$(find marm_description)/urdf/arm_base_gazebo.xacro" />
     <xacro:include filename="$(find marm_description)/urdf/marm.gazebo.urdf.xacro" />
-    <xacro:include filename="$(find marm_description)/urdf/kinect_gazebo.xacro" />
+    <!--xacro:include filename="$(find marm_description)/urdf/kinect_gazebo.xacro" /-->
     <mbot_base_gazebo/>
-    <link name="base_link">
+    <!--link name="base_link">
         <visual>
 			<origin xyz=" 0 0 0.02"  rpy="0 0 0"/>
@@ -26,8 +26,8 @@
         </collision>
         <box_inertial_matrix m="1000" w="1" h="0.02" d="1"/>
-    </link>
+    </link-->
 <!-- left_arm -->
     <joint name="base_stand_joint1" type="fixed">
-        <origin xyz="0.2 0 ${stand_length/2+0.08}" rpy="0 0 0" />
+        <origin xyz="0 0.2 ${stand_length/2+0.08}" rpy="0 0 ${M_PI/2}" />
         <parent link="base_link"/>
         <child link="stand1" />
@@ -55,5 +55,5 @@
 <!-- right_arm -->
     <joint name="base_stand_joint2" type="fixed">
-        <origin xyz="-0.2 0 ${stand_length/2+0.08}" rpy="0 0 0" />
+        <origin xyz="0 -0.2 ${stand_length/2+0.08}" rpy="0 0 ${M_PI/2}" />
         <parent link="base_link"/>
         <child link="stand2" />

File: marm_description/urdf/mbot_base_gazebo.xacro (robot description, xacro)
@@ -3,15 +3,15 @@
     <!-- PROPERTY LIST -->
     <xacro:property name="M_PI" value="3.1415926"/>
-    <xacro:property name="base_mass"   value="20" />
-    <xacro:property name="base_radius" value="0.20"/>
+    <xacro:property name="base_mass"   value="40" />
+    <xacro:property name="base_radius" value="0.40"/>
     <xacro:property name="base_length" value="0.16"/>
     <xacro:property name="wheel_mass"   value="2" />
     <xacro:property name="wheel_radius" value="0.06"/>
     <xacro:property name="wheel_length" value="0.025"/>
-    <xacro:property name="wheel_joint_y" value="0.19"/>
+    <xacro:property name="wheel_joint_y" value="0.38"/>
     <xacro:property name="wheel_joint_z" value="0.05"/>
     <xacro:property name="caster_mass"    value="0.5" />
     <xacro:property name="caster_radius"  value="0.015"/> <!-- wheel_radius - ( base_length/2 - wheel_joint_z) -->
-    <xacro:property name="caster_joint_x" value="0.18"/>
+    <xacro:property name="caster_joint_x" value="0.36"/>
     <!-- Defining the colors used in this robot -->
     <material name="yellow">
@@ -72,8 +72,8 @@
             <type>transmission_interface/SimpleTransmission</type>
             <joint name="${prefix}_wheel_joint" >
-                <hardwareInterface>hardware_interface/EffortJointInterface</hardwareInterface>
+                <hardwareInterface>hardware_interface/PositionJointInterface</hardwareInterface>
             </joint>
             <actuator name="${prefix}_wheel_joint_motor">
-                <hardwareInterface>hardware_interface/EffortJointInterface</hardwareInterface>
+                <hardwareInterface>hardware_interface/PositionJointInterface</hardwareInterface>
                 <mechanicalReduction>1</mechanicalReduction>
             </actuator>
@@ -82,9 +82,9 @@
     <!-- Macro for robot caster -->
     <xacro:macro name="caster" params="prefix reflect">
-        <joint name="${prefix}_caster_joint" type="continuous">
+        <joint name="${prefix}_caster_joint" type="fixed">
             <origin xyz="${reflect*caster_joint_x} 0 ${-(base_length/2 + caster_radius)}" rpy="0 0 0"/>
             <parent link="base_link"/>
             <child link="${prefix}_caster_link"/>
-            <axis xyz="0 1 0"/>
+            <!--axis xyz="0 1 0"/-->
         </joint>
         <link name="${prefix}_caster_link">
@@ -109,5 +109,30 @@
     </xacro:macro>
     <xacro:macro name="mbot_base_gazebo">
+<!--        <link name="dummy">
+        </link>
+        <joint name="dummy_joint" type="fixed">
+           <parent link="dummy"/>
+           <child link="base_footprint"/>
+        </joint>
         <link name="base_footprint">
+           <inertial>
+                <mass value="0.0001" />
+                <origin xyz="0 0 0" />
+                <inertia ixx="0" ixy="0" ixz="0"
+                    iyy="0" iyz="0"
+                    izz="0" />
+            </inertial>
+            <visual>
+                <origin xyz="0 0 0" rpy="0 0 0" />
+                <geometry>
+                    <box size="0.001 0.001 0.001" />
+                </geometry>
+            </visual>
+        </link>
+        <gazebo reference="base_footprint">
+            <turnGravityOff>false</turnGravityOff>
+        </gazebo>-->
+        <link name="base_footprint"></link>
+        <!--<link name="base_footprint">
            <inertial>
                 <mass value="0.0001" />
@@ -126,5 +151,5 @@
         <gazebo reference="base_footprint">
             <turnGravityOff>false</turnGravityOff>
-        </gazebo>
+        </gazebo>-->
         <joint name="base_footprint_joint" type="fixed">
             <origin xyz="0 0 ${base_length/2 + caster_radius*2}" rpy="0 0 0" />
@@ -160,5 +185,5 @@
                 <rosDebugLevel>Debug</rosDebugLevel>
                 <publishWheelTF>true</publishWheelTF>
-                <robotNamespace>/</robotNamespace>
+                <robotNamespace>/mbot_base</robotNamespace>
                 <publishTf>1</publishTf>
                 <publishWheelJointState>true</publishWheelJointState>

Commit message: init upload

File: marm_description/urdf/marm.xacro (robot description, xacro)
@@ -15,22 +15,6 @@
     <xacro:property name="camera_offset_z" value="0" />
     <mbot_base_gazebo/>
-    <!--link name="base_link">
-        <visual>
-			<origin xyz=" 0 0 0.02"  rpy="0 0 0"/>
-			    <geometry>
-				   <box size="1 1 0.02" />
-			    </geometry>
-			<material name="Black" />
-        </visual>
-        <collision>
-            <origin xyz=" 0 0 0.02"  rpy="0 0 0"/>
-            <geometry>
-                <box size="1 1 0.02" />
-            </geometry>
-        </collision>
-        <box_inertial_matrix m="1000" w="1" h="0.02" d="1"/>
-    </link-->
 <!-- left_arm -->
-    <!--joint name="base_stand_joint1" type="fixed">
+    <joint name="base_stand_joint1" type="fixed">
         <origin xyz="0 0.2 ${stand_length/2+0.08}" rpy="0 0 ${M_PI/2}" />
         <parent link="base_link"/>
@@ -56,7 +40,7 @@
         <material>Gazebo/Gray</material>
     </gazebo>
-    <arm_base prefix="left" parent="stand1" xyz="0 0 0" rpy="${M_PI/2} 0 0"/-->
+    <arm_base prefix="left" parent="stand1" xyz="0 0 0" rpy="${M_PI/2} 0 0"/>
 <!-- right_arm -->
-    <!--joint name="base_stand_joint2" type="fixed">
+    <joint name="base_stand_joint2" type="fixed">
         <origin xyz="0 -0.2 ${stand_length/2+0.08}" rpy="0 0 ${M_PI/2}" />
         <parent link="base_link"/>
@@ -82,19 +66,19 @@
         <material>Gazebo/Gray</material>
     </gazebo>
-    <arm_base prefix="right" parent="stand2" xyz="0 0 0" rpy="${M_PI/2} 0 0"/-->
+    <arm_base prefix="right" parent="stand2" xyz="0 0 0" rpy="${M_PI/2} 0 0"/>
     <!-- leftCamera -->
-    <!--joint name="left_camera_joint" type="fixed">
+    <joint name="left_camera_joint" type="fixed">
         <origin xyz="${camera_offset_x} ${camera_offset_y} ${camera_offset_z}" rpy="${M_PI/2} 0 0" />
         <parent link="left_link6"/>
         <child link="left_camera_link"/>
     </joint>
-    <xacro:usb_camera prefix="left_camera"/-->
+    <xacro:usb_camera prefix="left_camera"/>
     <!-- rightCamera -->
-    <!--joint name="right_camera_joint" type="fixed">
+    <joint name="right_camera_joint" type="fixed">
         <origin xyz="${camera_offset_x} ${camera_offset_y} ${camera_offset_z}" rpy="${M_PI/2} 0 0" />
         <parent link="right_link6"/>
         <child link="right_camera_link"/>
     </joint>
-    <xacro:usb_camera prefix="right_camera"/-->
+    <xacro:usb_camera prefix="right_camera"/>
     <!-- Kinect -->
   <!--  <joint name="kinect_frame_joint" type="fixed">
@@ -103,4 +87,4 @@
         <child link="camera_link"/>
     </joint>
-    <xacro:kinect_camera prefix="camera"/> -->```
+    <xacro:kinect_camera prefix="camera"/> -->
 </robot>

File: marm_description/urdf/mbot_base_gazebo.xacro (robot description, xacro)
@@ -3,15 +3,15 @@
     <!-- PROPERTY LIST -->
     <xacro:property name="M_PI" value="3.1415926"/>
-    <xacro:property name="base_mass"   value="20" />
-    <xacro:property name="base_radius" value="0.20"/>
+    <xacro:property name="base_mass"   value="40" />
+    <xacro:property name="base_radius" value="0.40"/>
     <xacro:property name="base_length" value="0.16"/>
     <xacro:property name="wheel_mass"   value="2" />
     <xacro:property name="wheel_radius" value="0.06"/>
     <xacro:property name="wheel_length" value="0.025"/>
-    <xacro:property name="wheel_joint_y" value="0.19"/>
+    <xacro:property name="wheel_joint_y" value="0.38"/>
     <xacro:property name="wheel_joint_z" value="0.05"/>
     <xacro:property name="caster_mass"    value="0.5" />
     <xacro:property name="caster_radius"  value="0.015"/> <!-- wheel_radius - ( base_length/2 - wheel_joint_z) -->
-    <xacro:property name="caster_joint_x" value="0.18"/>
+    <xacro:property name="caster_joint_x" value="0.36"/>
     <!-- Defining the colors used in this robot -->
     <material name="yellow">
@@ -72,8 +72,8 @@
             <type>transmission_interface/SimpleTransmission</type>
             <joint name="${prefix}_wheel_joint" >
-                <hardwareInterface>hardware_interface/PositionJointInterface</hardwareInterface>
+                <hardwareInterface>hardware_interface/EffortJointInterface</hardwareInterface>
             </joint>
             <actuator name="${prefix}_wheel_joint_motor">
-                <hardwareInterface>hardware_interface/PositionJointInterface</hardwareInterface>
+                <hardwareInterface>hardware_interface/EffortJointInterface</hardwareInterface>
                 <mechanicalReduction>1</mechanicalReduction>
             </actuator>
