Commit message: arm exception

File: marm_description/urdf/arm_base_gazebo.xacro (robot description, xacro)
@@ -32,5 +32,5 @@
     <xacro:property name="link3_length" value="0.15" />
     <xacro:property name="link3_mass" value="0.8" />
-    <!-- link4 properties -->
+    <!-- ink4 properties -->
     <xacro:property name="link4_radius" value="0.025" />
     <xacro:property name="link4_length" value="0.06" />
@@ -69,11 +69,11 @@
     </xacro:macro>
     <!-- /////////////////////////////////////   ARM BASE    ////////////////////////////////////////////// -->
-    <xacro:macro name="arm_base" params="parent xyz rpy">
-        <joint name="${parent}_arm_joint" type="fixed">
+    <xacro:macro name="arm_base" params="prefix parent xyz rpy">
+        <joint name="${prefix}_${parent}_arm_joint" type="fixed">
             <origin xyz="${xyz}" rpy="${rpy}" />
             <parent link="${parent}"/>
-            <child link="base_arm" />
-        </joint>
-        <link name="base_arm">
+            <child link="${prefix}_base_arm" />
+        </joint>
+        <link name="${prefix}_base_arm">
             <visual>
                 <origin xyz="0 0 0" rpy="0 0 0" />
@@ -83,11 +83,11 @@
             </visual>
         </link>
-        <joint name="base_joint" type="fixed">
+        <joint name="${prefix}_base_joint" type="fixed">
             <origin xyz="0 0 ${link0_length/2}" rpy="0 0 0" />
-            <parent link="base_arm"/>
-            <child link="link0" />
-        </joint>
-        <!-- /////////////////////////////////////    LINK0    ////////////////////////////////////////////// -->
-        <link name="link0">
+            <parent link="${prefix}_base_arm"/>
+            <child link="${prefix}_link0" />
+        </joint>
+        <!-- /////////////////////////////////////  link0    ////////////////////////////////////////////// -->
+        <link name="${prefix}_link0">
             <visual>
                 <origin xyz="0 0 0" rpy="0 0 0" />
@@ -105,13 +105,13 @@
             <cylinder_inertial_matrix m="${link0_mass}" r="${link0_radius}" h="${link0_length}"/>
         </link>
-        <joint name="joint1" type="revolute">
-            <parent link="link0"/>
-            <child link="link1"/>
+        <joint name="${prefix}_joint1" type="revolute">
+            <parent link="${prefix}_link0"/>
+            <child link="${prefix}_link1"/>
             <origin xyz="0 0 ${link0_length/2}" rpy="0 ${M_PI/2} 0" />
             <axis xyz="-1 0 0" />
             <limit effort="300" velocity="1" lower="${-M_PI}" upper="${M_PI}"/>
         </joint>
-        <!-- /////////////////////////////////////   LINK1  ////////////////////////////////////////////// -->
-        <link name="link1" >
+        <!-- /////////////////////////////////////   link1  ////////////////////////////////////////////// -->
+        <link name="${prefix}_link1" >
             <visual>
                 <origin xyz="-${link1_length/2} 0 0" rpy="0 ${M_PI/2} 0" />
@@ -129,13 +129,13 @@
             <cylinder_inertial_matrix m="${link1_mass}" r="${link1_radius}" h="${link1_length}"/>
         </link>
-        <joint name="joint2" type="revolute">
-            <parent link="link1"/>
-            <child link="link2"/>
+        <joint name="${prefix}_joint2" type="revolute">
+            <parent link="${prefix}_link1"/>
+            <child link="${prefix}_link2"/>
             <origin xyz="-${link1_length} 0 0.0" rpy="-${M_PI/2} 0 ${M_PI/2}" />
             <axis xyz="1 0 0" />
             <limit effort="300" velocity="1" lower="${-M_PI}" upper="${M_PI}" />
         </joint>
-        <!-- ///////////////////////////////////////   LINK2  ////////////////////////////////////////////// -->
-        <link name="link2" >
+        <!-- ///////////////////////////////////////   link2  ////////////////////////////////////////////// -->
+        <link name="${prefix}_link2" >
             <visual>
                 <origin xyz="0 0 ${link2_length/2}" rpy="0 0 0" />
@@ -153,13 +153,13 @@
             <cylinder_inertial_matrix m="${link2_mass}" r="${link2_radius}" h="${link2_length}"/>
         </link>
-        <joint name="joint3" type="revolute">
-            <parent link="link2"/>
-            <child link="link3"/>
+        <joint name="${prefix}_joint3" type="revolute">
+            <parent link="${prefix}_link2"/>
+            <child link="${prefix}_link3"/>
             <origin xyz="0 0 ${link2_length}" rpy="0 ${M_PI} 0" />
             <axis xyz="-1 0 0" />
             <limit effort="300" velocity="1" lower="${-M_PI}" upper="${M_PI}" />
         </joint>
-        <!-- /////////////////////////////////   LINK3  ///////////////////////////////////////////////////// -->
-        <link name="link3" >
+        <!-- /////////////////////////////////   link3  ///////////////////////////////////////////////////// -->
+        <link name="${prefix}_link3" >
             <visual>
                 <origin xyz="0 0 -${link3_length/2}" rpy="0 0 0" />
@@ -177,13 +177,13 @@
             <cylinder_inertial_matrix m="${link3_mass}" r="${link3_radius}" h="${link3_length}"/>
         </link>
-        <joint name="joint4" type="revolute">
-            <parent link="link3"/>
-            <child link="link4"/>
+        <joint name="${prefix}_joint4" type="revolute">
+            <parent link="${prefix}_link3"/>
+            <child link="${prefix}_link4"/>
             <origin xyz="0.0 0.0 -${link3_length}" rpy="0 ${M_PI/2} ${M_PI}" />
             <axis xyz="1 0 0" />
             <limit effort="300" velocity="1" lower="${-M_PI}" upper="${M_PI}" />
         </joint>
-        <!-- ///////////////////////////////////   LINK4  //////////////////////////////////////////////// -->
-        <link name="link4" >
+        <!-- ///////////////////////////////////   link4  //////////////////////////////////////////////// -->
+        <link name="${prefix}_link4" >
             <visual>
                 <origin xyz="${link4_length/2} 0 0" rpy="0 ${M_PI/2} 0" />
@@ -201,13 +201,13 @@
             <cylinder_inertial_matrix m="${link4_mass}" r="${link4_radius}" h="${link4_length}"/>
         </link>
-        <joint name="joint5" type="revolute">
-            <parent link="link4"/>
-            <child link="link5"/>
+        <joint name="${prefix}_joint5" type="revolute">
+            <parent link="${prefix}_link4"/>
+            <child link="${prefix}_link5"/>
             <origin xyz="${link4_length} 0.0 0.0" rpy="0 ${M_PI/2} 0" />
             <axis xyz="1 0 0" />
             <limit effort="300" velocity="1" lower="${-M_PI}" upper="${M_PI}" />
         </joint>
-        <!-- //////////////////////////////////   LINK5  ///////////////////////////////////////////////// -->
-        <link name="link5">
+        <!-- //////////////////////////////////   link5  ///////////////////////////////////////////////// -->
+        <link name="${prefix}_link5">
             <visual>
                 <origin xyz="0 0 ${link4_length/2}" rpy="0 0 0" />
@@ -225,13 +225,13 @@
             <cylinder_inertial_matrix m="${link5_mass}" r="${link5_radius}" h="${link5_length}"/>
         </link>
-        <joint name="joint6" type="revolute">
-            <parent link="link5"/>
-            <child link="link6"/>
+        <joint name="${prefix}_joint6" type="revolute">
+            <parent link="${prefix}_link5"/>
+            <child link="${prefix}_link6"/>
             <origin xyz="0 0 ${link4_length}" rpy="${1.5*M_PI} -${M_PI/2} 0" />
             <axis xyz="1 0 0" />
             <limit effort="300" velocity="1" lower="${-2*M_PI}" upper="${2*M_PI}" />
         </joint>
-        <!-- ////////////////////////////////   LINK6  ///////////////////////////////////////////////// -->
-        <link name="link6">
+        <!-- ////////////////////////////////   link6  ///////////////////////////////////////////////// -->
+        <link name="${prefix}_link6">
             <visual>
                 <origin xyz="${link6_length/2} 0 0 " rpy="0 ${M_PI/2} 0" />
@@ -249,7 +249,7 @@
             <cylinder_inertial_matrix m="${link6_mass}" r="${link6_radius}" h="${link6_length}"/>
         </link>
-        <joint name="finger_joint1" type="prismatic">
-            <parent link="link6"/>
-            <child link="gripper_finger_link1"/>
+        <joint name="${prefix}_finger_joint1" type="prismatic">
+            <parent link="${prefix}_link6"/>
+            <child link="${prefix}_gripper_finger_link1"/>
             <origin xyz="${link6_length} -0.03 0" rpy="0 0 0" />
             <axis xyz="0 1 0" />
@@ -258,5 +258,5 @@
         <!-- //////////////////////////////////////   gripper   ////////////////////////////////////////////// -->
         <!-- LEFT GRIPPER AFT LINK -->
-        <link name="gripper_finger_link1">
+        <link name="${prefix}_gripper_finger_link1">
             <visual>
                 <origin xyz="${gripper_height/2} 0 0" rpy="0 ${M_PI/2} 0" />
@@ -274,11 +274,11 @@
             <box_inertial_matrix m="${gripper_mass}" w="${gripper_width}" h="${gripper_height}" d="${gripper_length}"/>
         </link>
-        <joint name="finger_joint2" type="fixed">
-            <parent link="link6"/>
-            <child link="gripper_finger_link2"/>
+        <joint name="${prefix}_finger_joint2" type="fixed">
+            <parent link="${prefix}_link6"/>
+            <child link="${prefix}_gripper_finger_link2"/>
             <origin xyz="${link6_length} 0.03 0" rpy="0 0 0" />
         </joint>
         <!-- RIGHT GRIPPER AFT LINK -->
-        <link name="gripper_finger_link2">
+        <link name="${prefix}_gripper_finger_link2">
             <visual>
                 <origin xyz="${gripper_height/2} 0 0" rpy="0 ${M_PI/2} 0" />
@@ -297,39 +297,39 @@
         </link>
         <!-- Grasping frame -->
-        <link name="grasping_frame"/>
-        <joint name="grasping_frame_joint" type="fixed">
-            <parent link="link6"/>
-            <child link="grasping_frame"/>
+        <link name="${prefix}_grasping_frame"/>
+        <joint name="${prefix}_grasping_frame_joint" type="fixed">
+            <parent link="${prefix}_link6"/>
+            <child link="${prefix}_grasping_frame"/>
             <origin xyz="${gripper_height} 0 0" rpy="0 0 0"/>
         </joint>
         <!-- /////////////////////////////////   Gazebo   ////////////////////////////////////// -->
-        <gazebo reference="bottom_link">
-            <material>Gazebo/White</material>
-        </gazebo>
-        <gazebo reference="base_arm">
-            <material>Gazebo/White</material>
-        </gazebo>
-        <gazebo reference="link1">
+        <gazebo reference="${prefix}_bottom_link">
+            <material>Gazebo/White</material>
+        </gazebo>
+        <gazebo reference="${prefix}_base_arm">
+            <material>Gazebo/White</material>
+        </gazebo>
+        <gazebo reference="${prefix}_link1">
             <material>Gazebo/Blue</material>
         </gazebo>
-        <gazebo reference="link2">
-            <material>Gazebo/White</material>
-        </gazebo>
-        <gazebo reference="link3">
+        <gazebo reference="${prefix}_link2">
+            <material>Gazebo/White</material>
+        </gazebo>
+        <gazebo reference="${prefix}_link3">
             <material>Gazebo/Blue</material>
         </gazebo>
-        <gazebo reference="link4">
+        <gazebo reference="${prefix}_link4">
             <material>Gazebo/Black</material>
         </gazebo>
-        <gazebo reference="link5">
-            <material>Gazebo/White</material>
-        </gazebo>
-        <gazebo reference="link6">
+        <gazebo reference="${prefix}_link5">
+            <material>Gazebo/White</material>
+        </gazebo>
+        <gazebo reference="${prefix}_link6">
             <material>Gazebo/Blue</material>
         </gazebo>
-        <gazebo reference="gripper_finger_link1">
-            <material>Gazebo/White</material>
-        </gazebo>
-        <gazebo reference="gripper_finger_link2">
+        <gazebo reference="${prefix}_gripper_finger_link1">
+            <material>Gazebo/White</material>
+        </gazebo>
+        <gazebo reference="${prefix}_gripper_finger_link2">
             <material>Gazebo/White</material>
         </gazebo>
@@ -347,17 +347,11 @@
             </transmission>
         </xacro:macro>
-        <xacro:transmission_block joint_name="joint1"/>
-        <xacro:transmission_block joint_name="joint2"/>
-        <xacro:transmission_block joint_name="joint3"/>
-        <xacro:transmission_block joint_name="joint4"/>
-        <xacro:transmission_block joint_name="joint5"/>
-        <xacro:transmission_block joint_name="joint6"/>
-        <xacro:transmission_block joint_name="finger_joint1"/>
-        <!-- ros_control plugin -->
-        <gazebo>
-            <plugin name="gazebo_ros_control" filename="libgazebo_ros_control.so">
-                <robotNamespace>/arm2</robotNamespace>
-            </plugin>
-        </gazebo>
+        <xacro:transmission_block joint_name="${prefix}_joint1"/>
+        <xacro:transmission_block joint_name="${prefix}_joint2"/>
+        <xacro:transmission_block joint_name="${prefix}_joint3"/>
+        <xacro:transmission_block joint_name="${prefix}_joint4"/>
+        <xacro:transmission_block joint_name="${prefix}_joint5"/>
+        <xacro:transmission_block joint_name="${prefix}_joint6"/>
+        <xacro:transmission_block joint_name="${prefix}_finger_joint1"/>
     </xacro:macro>
 </robot>

File: marm_description/urdf/dual_arm.xacro (robot description, xacro)
@@ -1,14 +1,7 @@
 <?xml version="1.0"?>
-<robot name="arm" xmlns:xacro="http://www.ros.org/wiki/xacro">
+<robot xmlns:xacro="http://ros.org/wiki/xacro">
     <xacro:property name="stand_mass"   value="2" />
     <xacro:property name="stand_radius" value="0.03"/>
     <xacro:property name="stand_length" value="0.4"/>
-    <xacro:property name="kinect_offset_z" value="0.24" />
-    <xacro:property name="kinect_offset_p" value="0.4" />
-    <xacro:include filename="$(find marm_description)/urdf/mbot_base_gazebo.xacro" />
-    <xacro:include filename="$(find marm_description)/urdf/arm_base_gazebo.xacro" />
-    <xacro:include filename="$(find marm_description)/urdf/marm.gazebo.urdf.xacro" />
-    <xacro:include filename="$(find marm_description)/urdf/kinect_gazebo.xacro" />
-    <mbot_base_gazebo/>
 <!-- left_arm -->
     <joint name="base_stand_joint1" type="fixed">
@@ -63,10 +56,9 @@
     </gazebo>
     <arm_base prefix="right" parent="stand2" xyz="0 0 0" rpy="${M_PI/2} 0 0"/>
-    <!-- Kinect -->
-  <!--  <joint name="kinect_frame_joint" type="fixed">
-        <origin xyz="0 0 ${kinect_offset_z}" rpy="0 ${kinect_offset_p} 0" />
-        <parent link="stand1"/>
-        <child link="camera_link"/>
-    </joint>
-    <xacro:kinect_camera prefix="camera"/> -->
+   <!-- ros_control plugin -->
+     <gazebo>
+        <plugin name="${prefix}_gazebo_ros_control" filename="libgazebo_ros_control.so">
+            <robotNamespace>/arm2</robotNamespace>
+        </plugin>
+    </gazebo>
 </robot>

File: marm_description/urdf/mbot_base_gazebo.xacro (robot description, xacro)
@@ -4,14 +4,14 @@
     <xacro:property name="M_PI" value="3.1415926"/>
     <xacro:property name="base_mass"   value="20" />
-    <xacro:property name="base_radius" value="0.20"/>
+    <xacro:property name="base_radius" value="0.40"/>
     <xacro:property name="base_length" value="0.16"/>
     <xacro:property name="wheel_mass"   value="2" />
     <xacro:property name="wheel_radius" value="0.06"/>
     <xacro:property name="wheel_length" value="0.025"/>
-    <xacro:property name="wheel_joint_y" value="0.19"/>
+    <xacro:property name="wheel_joint_y" value="0.38"/>
     <xacro:property name="wheel_joint_z" value="0.05"/>
     <xacro:property name="caster_mass"    value="0.5" />
     <xacro:property name="caster_radius"  value="0.015"/> <!-- wheel_radius - ( base_length/2 - wheel_joint_z) -->
-    <xacro:property name="caster_joint_x" value="0.18"/>
+    <xacro:property name="caster_joint_x" value="0.36"/>
     <!-- Defining the colors used in this robot -->
     <material name="yellow">
@@ -109,11 +109,17 @@
     </xacro:macro>
     <xacro:macro name="mbot_base_gazebo">
+<!--        <link name="dummy">
+        </link>
+        <joint name="dummy_joint" type="fixed">
+           <parent link="dummy"/>
+           <child link="base_footprint"/>
+        </joint>
         <link name="base_footprint">
            <inertial>
                 <mass value="0.0001" />
                 <origin xyz="0 0 0" />
-                <inertia ixx="0.0001" ixy="0.0" ixz="0.0"
-                    iyy="0.0001" iyz="0.0"
-                    izz="0.0001" />
+                <inertia ixx="0" ixy="0" ixz="0"
+                    iyy="0" iyz="0"
+                    izz="0" />
             </inertial>
             <visual>
@@ -126,5 +132,6 @@
         <gazebo reference="base_footprint">
             <turnGravityOff>false</turnGravityOff>
-        </gazebo>
+        </gazebo>-->
+        <link name="base_footprint"></link>
         <joint name="base_footprint_joint" type="fixed">
             <origin xyz="0 0 ${base_length/2 + caster_radius*2}" rpy="0 0 0" />
@@ -160,5 +167,5 @@
                 <rosDebugLevel>Debug</rosDebugLevel>
                 <publishWheelTF>true</publishWheelTF>
-                <robotNamespace>/</robotNamespace>
+                <robotNamespace>/mbot_base</robotNamespace>
                 <publishTf>1</publishTf>
                 <publishWheelJointState>true</publishWheelJointState>

Commit message: nothing

File: marm_description/urdf/arm_base_gazebo.xacro (robot description, xacro)
@@ -339,8 +339,8 @@
                 <type>transmission_interface/SimpleTransmission</type>
                 <joint name="${joint_name}">
-                    <hardwareInterface>hardware_interface/EffortJointInterface</hardwareInterface>
+                    <hardwareInterface>EffortJointInterface</hardwareInterface>
                 </joint>
                 <actuator name="${joint_name}_motor">
-                    <hardwareInterface>hardware_interface/EffortJointInterface</hardwareInterface>
+                    <hardwareInterface>EffortJointInterface</hardwareInterface>
                     <mechanicalReduction>1</mechanicalReduction>
                 </actuator>

File: marm_description/urdf/mbot_base_gazebo.xacro (robot description, xacro)
@@ -134,4 +134,22 @@
         </gazebo>-->
         <link name="base_footprint"></link>
+        <!--<link name="base_footprint">
+           <inertial>
+                <mass value="0.0001" />
+                <origin xyz="0 0 0" />
+                <inertia ixx="0.0001" ixy="0.0" ixz="0.0"
+                    iyy="0.0001" iyz="0.0"
+                    izz="0.0001" />
+            </inertial>
+            <visual>
+                <origin xyz="0 0 0" rpy="0 0 0" />
+                <geometry>
+                    <box size="0.001 0.001 0.001" />
+                </geometry>
+            </visual>
+        </link>
+        <gazebo reference="base_footprint">
+            <turnGravityOff>false</turnGravityOff>
+        </gazebo>-->
         <joint name="base_footprint_joint" type="fixed">
             <origin xyz="0 0 ${base_length/2 + caster_radius*2}" rpy="0 0 0" />

File: marm_description/urdf/mbot_with_arm_kinect_gazebo.xacro (robot description, xacro)
@@ -1,4 +1,4 @@
 <?xml version="1.0"?>
-<robot name="arm" xmlns:xacro="http://www.ros.org/wiki/xacro">
+<robot name="marm" xmlns:xacro="http://www.ros.org/wiki/xacro">
     <xacro:property name="stand_mass"   value="2" />
     <xacro:property name="stand_radius" value="0.03"/>

Commit message: holy shit

File: marm_description/urdf/arm_base_gazebo.xacro (robot description, xacro)
@@ -339,8 +339,8 @@
                 <type>transmission_interface/SimpleTransmission</type>
                 <joint name="${joint_name}">
-                    <hardwareInterface>EffortJointInterface</hardwareInterface>
+                    <hardwareInterface>hardware_interface/EffortJointInterface</hardwareInterface>
                 </joint>
                 <actuator name="${joint_name}_motor">
-                    <hardwareInterface>EffortJointInterface</hardwareInterface>
+                    <hardwareInterface>hardware_interface/EffortJointInterface</hardwareInterface>
                     <mechanicalReduction>1</mechanicalReduction>
                 </actuator>

File: marm_description/urdf/mbot_base_gazebo.xacro (robot description, xacro)
@@ -181,5 +181,5 @@
         <caster prefix="back"  reflect="1"/>
         <!-- controller -->
-        <gazebo>
+        <!--<gazebo>
             <plugin name="differential_drive_controller" filename="libgazebo_ros_diff_drive.so">
                 <rosDebugLevel>Debug</rosDebugLevel>
@@ -203,5 +203,5 @@
                 <robotBaseFrame>base_footprint</robotBaseFrame>
             </plugin>
-        </gazebo>
+        </gazebo> -->
     </xacro:macro>
 </robot>

File: marm_description/urdf/mbot_with_arm_kinect_gazebo.xacro (robot description, xacro)
@@ -6,9 +6,25 @@
     <xacro:property name="kinect_offset_z" value="0.24" />
     <xacro:property name="kinect_offset_p" value="0.4" />
-    <xacro:include filename="$(find marm_description)/urdf/mbot_base_gazebo.xacro" />
+<!--    <xacro:include filename="$(find marm_description)/urdf/mbot_base_gazebo.xacro" />-->
     <xacro:include filename="$(find marm_description)/urdf/arm_base_gazebo.xacro" />
     <xacro:include filename="$(find marm_description)/urdf/marm.gazebo.urdf.xacro" />
     <xacro:include filename="$(find marm_description)/urdf/kinect_gazebo.xacro" />
-    <mbot_base_gazebo/>
+<!--    <mbot_base_gazebo/> -->
+    <link name="base_link">
+        <visual>
+			<origin xyz=" 0 0 0.02"  rpy="0 0 0"/>
+			    <geometry>
+				   <box size="1 1 0.02" />
+			    </geometry>
+			<material name="Black" />
+        </visual>
+        <collision>
+            <origin xyz=" 0 0 0.02"  rpy="0 0 0"/>
+            <geometry>
+                <box size="1 1 0.02" />
+            </geometry>
+        </collision>
+        <box_inertial_matrix m="1000" w="1" h="0.02" d="1"/>
+    </link>
 <!-- left_arm -->
     <joint name="base_stand_joint1" type="fixed">
